File: dev_f070.sch (KiCad schematic (older format))
At the start: 22 parts

Commit message: update schem
Parts:
- added J?: Left_Headers, Connector_PinHeader_2.54mm:PinHeader_1x07_P2.54mm_Vertical, symbol Connector:Conn_01x07_Male
- added J?: Right_Headers, Connector_PinHeader_2.54mm:PinHeader_1x08_P2.54mm_Vertical, symbol Connector:Conn_01x08_Male
- C? (x3): footprint (none) -> Capacitor_SMD:C_1210_3225Metric
- C?: footprint (none) -> Capacitor_SMD:C_1206_3216Metric
- Y?: footprint (none) -> Crystal:Resonator_SMD_muRata_SFECV-3Pin_6.9x2.9mm_HandSoldering
Connections:
- net LedB: now also J?.6 (Pin_6)
- net LedG: now also J?.5 (Pin_5)
- net LedR: now also J?.4 (Pin_4)
- net PA0: now also J?.3 (Pin_3)
- net PA10|12: now also J?.3 (Pin_3)
- net PA13: now also J?.2 (Pin_2)
- net PA14: now also J?.1 (Pin_1)
- net PA4: now also J?.7 (Pin_7)
- net PA5: now also J?.8 (Pin_8)
- net PA6: now also J?.7 (Pin_7)
- net PA7: now also J?.6 (Pin_6)
- net PA9|11: now also J?.4 (Pin_4)
- net Q1: now also J?.1 (Pin_1)
- net Q2: now also J?.2 (Pin_2)
- net PB1: now reaches U?.14 (PB1)
- net PB1: now also J?.5 (Pin_5)
Changed lines of the file:
@@
 EESchema Schematic File Version 4
+LIBS:dev_f070-cache
 EELAYER 30 0
 EELAYER END
@@
 F 0 "C?" H 6965 1246 50  0000 L CNN
 F 1 "10uF" H 6965 1155 50  0000 L CNN
-F 2 "" H 6888 1050 50  0001 C CNN
+F 2 "Capacitor_SMD:C_1210_3225Metric" H 6888 1050 50  0001 C CNN
 F 3 "~" H 6850 1200 50  0001 C CNN
 	1    6850 1200
@@
 F 0 "C?" H 8315 1246 50  0000 L CNN
 F 1 "1uF" H 8315 1155 50  0000 L CNN
-F 2 "" H 8238 1050 50  0001 C CNN
+F 2 "Capacitor_SMD:C_1210_3225Metric" H 8238 1050 50  0001 C CNN
 F 3 "~" H 8200 1200 50  0001 C CNN
 	1    8200 1200
@@
 F 0 "Y?" H 3000 2698 50  0000 C CNN
 F 1 "Resonator" H 3000 2607 50  0000 C CNN
-F 2 "" H 2975 2450 50  0001 C CNN
+F 2 "Crystal:Resonator_SMD_muRata_SFECV-3Pin_6.9x2.9mm_HandSoldering" H 2975 2450 50  0001 C CNN
 F 3 "~" H 2975 2450 50  0001 C CNN
 	1    3000 2450
@@
 F 0 "C?" V 5652 1200 50  0000 C CNN
 F 1 "10uF" V 5561 1200 50  0000 C CNN
-F 2 "" H 5438 1050 50  0001 C CNN
+F 2 "Capacitor_SMD:C_1210_3225Metric" H 5438 1050 50  0001 C CNN
 F 3 "~" H 5400 1200 50  0001 C CNN
 	1    5400 1200
@@
 F 0 "C?" V 5148 1400 50  0000 C CNN
 F 1 "100pF" V 5239 1400 50  0000 C CNN
-F 2 "" H 5438 1250 50  0001 C CNN
+F 2 "Capacitor_SMD:C_1206_3216Metric" H 5438 1250 50  0001 C CNN
 F 3 "~" H 5400 1400 50  0001 C CNN
 	1    5400 1400
@@
 	1    0    0    -1
 $EndComp
+$Comp
+L Connector:Conn_01x07_Male J?
+U 1 1 5E2EEC2E
+P 3950 4950
+F 0 "J?" H 4058 5431 50  0000 C CNN
+F 1 "Left_Headers" H 4058 5340 50  0000 C CNN
+F 2 "Connector_PinHeader_2.54mm:PinHeader_1x07_P2.54mm_Vertical" H 3950 4950 50  0001 C CNN
+F 3 "~" H 3950 4950 50  0001 C CNN
+	1    3950 4950
+	1    0    0    -1
+$EndComp
+$Comp
+L Connector:Conn_01x08_Male J?
+U 1 1 5E2F1CDD
+P 6350 4900
+F 0 "J?" H 6458 5381 50  0000 C CNN
+F 1 "Right_Headers" H 6458 5290 50  0000 C CNN
+F 2 "Connector_PinHeader_2.54mm:PinHeader_1x08_P2.54mm_Vertical" H 6350 4900 50  0001 C CNN
+F 3 "~" H 6350 4900 50  0001 C CNN
+	1    6350 4900
+	1    0    0    -1
+$EndComp
+Text GLabel 4150 4650 2    50   Output ~ 0
+Q1
+Text GLabel 4150 4750 2    50   Output ~ 0
+Q2
+Text GLabel 4150 4850 2    50   Output ~ 0
+PA0
+Text GLabel 4150 4950 2    50   Output ~ 0
+PA1
+Text GLabel 4150 5050 2    50   Output ~ 0
+PA2
+Text GLabel 4150 5150 2    50   Output ~ 0
+PA3
+Text GLabel 4150 5250 2    50   Output ~ 0
+PA4
+Text GLabel 6550 4600 2    50   Output ~ 0
+PA14
+Text GLabel 6550 4700 2    50   Output ~ 0
+PA13
+Text GLabel 6550 4800 2    50   Output ~ 0
+PA10|12
+Text GLabel 6550 4900 2    50   Output ~ 0
+PA9|11
+Text GLabel 4650 3000 0    50   Input ~ 0
+PB1
+Text GLabel 6550 5000 2    50   Output ~ 0
+PB1
+Text GLabel 6550 5100 2    50   Output ~ 0
+PA7
+Text GLabel 6550 5200 2    50   Output ~ 0
+PA6
+Text GLabel 6550 5300 2    50   Output ~ 0
+PA5
 $EndSCHEMATC
